Commit message: updated URDF

File: URDF_Files/spider-viz/urdf/spider-viz.urdf (robot description, URDF)
Before this commit: robot spider-viz, 9 links, 8 joints
Links:
- link Leg_lower_3: mass 0.00601286144806057 -> 0.00601286144806056
- link Leg_lower_4: mass 0.00601286144806057 -> 0.00601286144806056
- link Leg_upper_1: mass 0.0300293935761664 -> 0.0300293941663224
- link Leg_upper_2: mass 0.0300293937966342 -> 0.0300293937574502
- link Leg_upper_3: mass 0.0300293927667882 -> 0.0300293941663224
- link Leg_upper_4: mass 0.0300293936383057 -> 0.0300293937574502
Joints:
- joint Leg_lower_3: origin xyz=0.055094 0.01315 0 rpy=2.1537 -1.5708 0 -> xyz=0.0550943670538193 0.0131500000000001 0 rpy=2.15366156766054 -1.5707963267949 0
- joint Leg_lower_4: origin xyz=0.055094 0.01315 0 rpy=2.015 -1.5708 0 -> xyz=0.0550943670538193 0.0131500000000001 0 rpy=2.01503172708615 -1.5707963267949 0
- joint Leg_upper_4: origin xyz=0.055831 -0.023773 0.032257 rpy=1.5708 0 0.80024 -> xyz=0.0558314237945949 -0.0237725392912401 0.0322574126580795 rpy=1.5707963267949 0 0.800237564975585

Commit message: stuff

File: URDF_Files/spider-viz/urdf/spider-viz.urdf (robot description, URDF)
Before this commit: robot spider-viz, 9 links, 8 joints
Links:
- link base_link: mass 0.0921702413076556 -> 0.0921702413076557
Joints:
- joint Leg_lower_1: limit (none) -> lower=0 upper=0 effort=0 velocity=0; origin xyz=0.0550943670538194 0.0131500000000004 0 rpy=-0.181875741727454 -1.57079631189374 -0.949890242088311 -> xyz=0.055094 0.01315 0 rpy=-0.18188 -1.5708 -0.94989; type continuous -> revolute
- joint Leg_lower_2: limit (none) -> lower=0 upper=0 effort=0 velocity=0; origin xyz=0.0550943670538194 0.0131500000000001 0 rpy=-1.43048154935128 -1.57079631189374 0.320209415436932 -> xyz=0.055094 0.01315 0 rpy=-1.4305 -1.5708 0.32021; type continuous -> revolute
- joint Leg_lower_3: limit (none) -> lower=0 upper=0 effort=0 velocity=0; origin xyz=0.0550943670538193 0.0131500000000001 0 rpy=2.15366156766054 -1.5707963267949 0 -> xyz=0.055094 0.01315 0 rpy=2.1537 -1.5708 0; type continuous -> revolute
- joint Leg_lower_4: limit (none) -> lower=0 upper=0 effort=0 velocity=0; origin xyz=0.0550943670538193 0.0131500000000001 0 rpy=2.01503172708615 -1.5707963267949 0 -> xyz=0.055094 0.01315 0 rpy=2.015 -1.5708 0; type continuous -> revolute
- joint Leg_upper_1: limit (none) -> lower=0 upper=0 effort=0 velocity=0; origin xyz=0.0558314237945942 -0.082056810538703 0.032257412658079 rpy=1.5707963267949 0 -0.770351507810951 -> xyz=0.055831 -0.082057 0.032257 rpy=1.5708 0 -0.77035; type continuous -> revolute
- joint Leg_upper_2: limit (none) -> lower=0 upper=0 effort=0 velocity=0; origin xyz=-0.00245284745286578 -0.0820568105387026 0.0322574126580794 rpy=1.5707963267949 0 -2.34833207396482 -> xyz=-0.0024528 -0.082057 0.032257 rpy=1.5708 0 -2.3483; type continuous -> revolute
- joint Leg_upper_3: limit (none) -> lower=0 upper=0 effort=0 velocity=0; origin xyz=-0.00245284745286686 -0.0237725392912402 0.0322574126580794 rpy=1.5707963267949 0 2.44535194984567 -> xyz=-0.0024528 -0.023773 0.032257 rpy=1.5708 0 2.4454; type continuous -> revolute
- joint Leg_upper_4: limit (none) -> lower=0 upper=0 effort=0 velocity=0; origin xyz=0.0558314237945949 -0.0237725392912401 0.0322574126580795 rpy=1.5707963267949 0 0.800237564975585 -> xyz=0.055831 -0.023773 0.032257 rpy=1.5708 0 0.80024; type continuous -> revolute

Commit message: testing part instead of asm

File: URDF_Files/spider-viz/urdf/spider-viz.urdf (robot description, URDF)
Before this commit: robot spider-viz, 9 links, 8 joints
Links:
- removed link Leg_lower_1
- removed link Leg_lower_2
- removed link Leg_lower_3
- removed link Leg_lower_4
- removed link Leg_upper_1
- removed link Leg_upper_2
- removed link Leg_upper_3
- removed link Leg_upper_4
- added link lower_11, mass 0.005129; collision mesh filename=package://spider-viz/meshes/lower_11.STL; visual mesh filename=package://spider-viz/meshes/lower_11.STL
- added link lower_21, mass 0.005129; collision mesh filename=package://spider-viz/meshes/lower_21.STL; visual mesh filename=package://spider-viz/meshes/lower_21.STL
- added link lower_32, mass 0.00512899375178834; collision mesh filename=package://spider-viz/meshes/lower_32.STL; visual mesh filename=package://spider-viz/meshes/lower_32.STL
- added link lower_42, mass 0.005129; collision mesh filename=package://spider-viz/meshes/lower_42.STL; visual mesh filename=package://spider-viz/meshes/lower_42.STL
- added link upper_11, mass 0.014321; collision mesh filename=package://spider-viz/meshes/upper_11.STL; visual mesh filename=package://spider-viz/meshes/upper_11.STL
- added link upper_21, mass 0.0143208814059842; collision mesh filename=package://spider-viz/meshes/upper_21.STL; visual mesh filename=package://spider-viz/meshes/upper_21.STL
- added link upper_32, mass 0.014321; collision mesh filename=package://spider-viz/meshes/upper_32.STL; visual mesh filename=package://spider-viz/meshes/upper_32.STL
- added link upper_42, mass 0.014321; collision mesh filename=package://spider-viz/meshes/upper_42.STL; visual mesh filename=package://spider-viz/meshes/upper_42.STL
- link base_link: mass 0.0921702413076557 -> 0.0501529793920895
Joints:
- removed joint Leg_lower_1
- removed joint Leg_lower_2
- removed joint Leg_lower_3
- removed joint Leg_lower_4
- removed joint Leg_upper_1
- removed joint Leg_upper_2
- removed joint Leg_upper_3
- removed joint Leg_upper_4
- added joint lower_11: type continuous, parent upper_11, child lower_11, origin xyz=0.055094 0.01315 0 rpy=1.5708 -1.5708 0, axis 1 0 0
- added joint lower_21: type continuous, parent upper_21, child lower_21, origin xyz=0.0550000000000001 0.0131500000000001 0 rpy=1.5707963267949 -1.5707963267949 0, axis 1 0 0
- added joint lower_32: type continuous, parent upper_32, child lower_32, origin xyz=0.096308 0.06315 0.039113 rpy=1.5708 -1.5708 0, axis 1 0 0
- added joint lower_42: type continuous, parent upper_42, child lower_42, origin xyz=0.096308 -0.03685 0.048063 rpy=1.5708 -1.5708 0, axis 1 0 0
- added joint upper_11: type continuous, parent base_link, child upper_11, origin xyz=0.055831 -0.023773 0.032257 rpy=1.5708 0 0.7854, axis 0 1 0
- added joint upper_21: type continuous, parent base_link, child upper_21, origin xyz=-0.0024528 -0.082057 0.032257 rpy=1.5708 0 -2.3562, axis 0 1 0
- added joint upper_32: type continuous, parent base_link, child upper_32, origin xyz=0.0558314237945951 -0.0237725392912399 -0.0177425873419207 rpy=1.5707963267949 0 -0.785398163397447, axis 0 1 0
- added joint upper_42: type continuous, parent base_link, child upper_42, origin xyz=-0.0024528 -0.082057 0.082257 rpy=1.5708 0 2.3562, axis 0 1 0

Commit message: updated URDF files again, hopefully for the last time

File: URDF_Files/spider-viz/urdf/spider-viz.urdf (robot description, URDF)
Before this commit: robot spider-viz, 9 links, 8 joints
Links:
- link lower_11: mass 0.005129 -> 0.00512899375178834
- link lower_21: mass 0.005129 -> 0.00512899375178834
- link lower_42: mass 0.005129 -> 0.00512899375178834
- link upper_11: mass 0.014321 -> 0.0143208814059843
- link upper_32: mass 0.014321 -> 0.0143208810051291
- link upper_42: mass 0.014321 -> 0.0143208810051291
Joints:
- joint lower_11: origin xyz=0.055094 0.01315 0 rpy=1.5708 -1.5708 0 -> xyz=0.0550943670538194 0.0131500000000002 0 rpy=1.5707963267949 -1.5707963267949 0
- joint lower_32: origin xyz=0.096308 0.06315 0.039113 rpy=1.5708 -1.5708 0 -> xyz=0.0550943670538193 0.0131500000000003 -0.00210000000000139 rpy=1.5707963267949 -1.5707963267949 0
- joint lower_42: origin xyz=0.096308 -0.03685 0.048063 rpy=1.5708 -1.5708 0 -> xyz=0.0550943670538194 0.0131500000000001 0.00684999999999963 rpy=1.5707963267949 -1.5707963267949 0
- joint upper_11: origin xyz=0.055831 -0.023773 0.032257 rpy=1.5708 0 0.7854 -> xyz=0.055831423794595 -0.0237725392912399 0.0322574126580793 rpy=1.5707963267949 0 0.785398163397433
- joint upper_21: origin xyz=-0.0024528 -0.082057 0.032257 rpy=1.5708 0 -2.3562 -> xyz=-0.00245284745286621 -0.0820568105387026 0.0322574126580794 rpy=1.5707963267949 0 -2.35619449019236
- joint upper_32: origin xyz=0.0558314237945951 -0.0237725392912399 -0.0177425873419207 rpy=1.5707963267949 0 -0.785398163397447 -> xyz=0.0558314237945942 -0.082056810538703 0.032257412658079 rpy=1.5707963267949 0 -0.785398163397447
- joint upper_42: origin xyz=-0.0024528 -0.082057 0.082257 rpy=1.5708 0 2.3562 -> xyz=-0.00245284745286684 -0.0237725392912402 0.0322574126580794 rpy=1.5707963267949 0 2.35619449019235

Commit message: testing limits

File: URDF_Files/spider-viz/urdf/spider-viz.urdf (robot description, URDF)
Before this commit: robot spider-viz, 9 links, 8 joints
Links:
- link lower_11: mass 0.00512899375178834 -> 0.005129
- link lower_21: mass 0.00512899375178834 -> 0.005129
- link lower_32: mass 0.00512899375178834 -> 0.005129
- link lower_42: mass 0.00512899375178834 -> 0.005129
- link upper_11: mass 0.0143208814059843 -> 0.014321
- link upper_21: mass 0.0143208814059842 -> 0.014321
- link upper_32: mass 0.0143208810051291 -> 0.014321
- link upper_42: mass 0.0143208810051291 -> 0.014321
Joints:
- joint lower_11: origin xyz=0.0550943670538194 0.0131500000000002 0 rpy=1.5707963267949 -1.5707963267949 0 -> xyz=0.055094 0.01315 0 rpy=1.5708 -1.5708 0
- joint lower_32: origin xyz=0.0550943670538193 0.0131500000000003 -0.00210000000000139 rpy=1.5707963267949 -1.5707963267949 0 -> xyz=0.055094 0.01315 -0.0021 rpy=1.5708 -1.5708 0
- joint upper_11: limit (none) -> lower=-1.0472 upper=1.0472 effort=0 velocity=0; origin xyz=0.055831423794595 -0.0237725392912399 0.0322574126580793 rpy=1.5707963267949 0 0.785398163397433 -> xyz=0.055831 -0.023773 0.032257 rpy=1.5708 0 0.7854
- joint upper_21: limit (none) -> lower=-1.0472 upper=1.0472 effort=0 velocity=0; origin xyz=-0.00245284745286621 -0.0820568105387026 0.0322574126580794 rpy=1.5707963267949 0 -2.35619449019236 -> xyz=-0.0024528 -0.082057 0.032257 rpy=1.5708 0 -2.3562
- joint upper_32: limit (none) -> lower=-1.0472 upper=1.0472 effort=0 velocity=0; origin xyz=0.0558314237945942 -0.082056810538703 0.032257412658079 rpy=1.5707963267949 0 -0.785398163397447 -> xyz=0.055831 -0.082057 0.032257 rpy=1.5708 0 -0.7854
- joint upper_42: limit (none) -> lower=-1.0472 upper=1.0472 effort=0 velocity=0; origin xyz=-0.00245284745286684 -0.0237725392912402 0.0322574126580794 rpy=1.5707963267949 0 2.35619449019235 -> xyz=-0.0024528 -0.023773 0.032257 rpy=1.5708 0 2.3562

Commit message: manually updated URDF file for simplified sollision

File: URDF_Files/spider-viz/urdf/spider-viz.urdf (robot description, URDF)
Before this commit: robot spider-viz, 9 links, 8 joints
Links:
- link base_link: geometry collision box size=0.07 0.07 0.01; visual mesh filename=package://spider-viz/meshes/base_link.STL
- link lower_11: geometry collision box size=0.005 0.09 0.01; visual mesh filename=package://spider-viz/meshes/lower_11.STL
- link lower_21: geometry collision box size=0.005 0.09 0.01; visual mesh filename=package://spider-viz/meshes/lower_21.STL
- link lower_32: geometry collision box size=0.005 0.09 0.01; visual mesh filename=package://spider-viz/meshes/lower_32.STL
- link lower_42: geometry collision box size=0.005 0.09 0.01; visual mesh filename=package://spider-viz/meshes/lower_42.STL
- link upper_11: geometry collision box size=0.06 0.01 0.015; visual mesh filename=package://spider-viz/meshes/upper_11.STL
- link upper_21: geometry collision box size=0.06 0.01 0.015; visual mesh filename=package://spider-viz/meshes/upper_21.STL
- link upper_32: geometry collision box size=0.06 0.01 0.015; visual mesh filename=package://spider-viz/meshes/upper_32.STL
- link upper_42: geometry collision box size=0.06 0.01 0.015; visual mesh filename=package://spider-viz/meshes/upper_42.STL
