File: PCB/Spider_Upper/Spider_Upper.kicad_sch (KiCad schematic)
At the start: 21 parts, among them J16 Conn_01x02, J17 Conn_02x06_Odd_Even, J18 Conn_02x06_Odd_Even, J19 Conn_02x06_Odd_Even, J20 Conn_02x06_Odd_Even, U6 LM2675M-3.3

Commit message: finished V1 PCB
Parts:
- removed H1, H2, H3, H4: MountingHole, MountingHole:MountingHole_3.2mm_M3, symbol Mechanical:MountingHole
- removed U1, U2: ~, Adafruit ESPs:ESP32-C6, symbol Adafruit_ESP32:ESP32-C6
- removed U4: ~, Package_SO:TSSOP-16-1EP_4.4x5mm_P0.65mm, symbol Misc:TMUX4051PWR
- removed U6: LM2675M-3.3, Package_SO:SOIC-8_3.9x4.9mm_P1.27mm, symbol Regulator_Switching:LM2675M-3.3
- added C1, C10, C12, C14, C15, C16, C17, C3, C5: 0.1u, Capacitor_SMD:C_0603_1608Metric_Pad1.08x0.95mm_HandSolder, symbol Device:C
- added C11: 100nF, Capacitor_SMD:C_0805_2012Metric, symbol Device:C
- added C13: 10uF, Capacitor_SMD:C_0805_2012Metric, symbol Device:C
- added C2, C9: 10u, Capacitor_SMD:C_0603_1608Metric_Pad1.08x0.95mm_HandSolder, symbol Device:C
- added D2, D3, D4, D5: LED, LED_SMD:LED_0805_2012Metric_Pad1.15x1.40mm_HandSolder, symbol Device:LED
- added J6, J7: USB_C_Receptacle_USB2.0, Connector_USB:USB_C_Receptacle_JAE_DX07S016JA1R1500, symbol Connector:USB_C_Receptacle_USB2.0
- added J8, J9: Conn_01x05, Connector_PinHeader_2.54mm:PinHeader_1x05_P2.54mm_Vertical, symbol Connector_Generic:Conn_01x05
- added Q1, Q2, Q3, Q4: DNBT8105-7, Package_TO_SOT_SMD:SOT-23, symbol Device:Q_NPN_BEC
- added R1, R2, R3, R4: 27, Resistor_SMD:R_0603_1608Metric_Pad0.98x0.95mm_HandSolder, symbol Device:R
- added R10, R12, R13, R9: 5.1k, Resistor_SMD:R_0603_1608Metric_Pad0.98x0.95mm_HandSolder, symbol Device:R
- added R11, R20, R21, R25, R26, R5: 10k, Resistor_SMD:R_0603_1608Metric_Pad0.98x0.95mm_HandSolder, symbol Device:R
- added R14, R15, R16: 280, Resistor_SMD:R_0603_1608Metric_Pad0.98x0.95mm_HandSolder, symbol Device:R
- added R17, R19, R22, R23, R24, R7, R8: 2.2k, Resistor_SMD:R_0603_1608Metric_Pad0.98x0.95mm_HandSolder, symbol Device:R
- added R18: 180, Resistor_SMD:R_0603_1608Metric_Pad0.98x0.95mm_HandSolder, symbol Device:R
- added SW1, SW2, SW3, SW4: SW_SPST, Button_Switch_SMD:SW_SPST_B3U-1000P, symbol Switch:SW_SPST
- added U1, U3: FT231XS, Package_SO:SSOP-20_3.9x8.7mm_P0.635mm, symbol Interface_USB:FT231XS
- added U4, U7: ESP32-C6-WROOM-1, Espressif:ESP32-C6-WROOM-1, symbol Espressif:ESP32-C6-WROOM-1
- added U5: LM2675M-5, Package_SO:SOIC-8_3.9x4.9mm_P1.27mm, symbol Regulator_Switching:LM2675M-5
- added U6: LD1117S33TR_SOT223, Package_TO_SOT_SMD:SOT-223-3_TabPin2, symbol Regulator_Linear:LD1117S33TR_SOT223
- added U8: ~, Package_SO:TSSOP-16-1EP_4.4x5mm_P0.65mm, symbol Misc:PCA9534PWR
- C4: value 10uF -> 0.1u; footprint Capacitor_SMD:C_0805_2012Metric -> Capacitor_SMD:C_0603_1608Metric_Pad1.08x0.95mm_HandSolder
- renumbered C1 to C6, C2 to C7, C3 to C8, J20 to J?, J16 to J?, J18 to J?, J17 to J?, J19 to J?, R1 to R6, U5 to U2
Connections:
- net +12V: now also U5.7 (VIN)
- net +3.3V: now also C4.1, C1.1, C10.1, C13.1, C2.1, C3.1, C9.1, J8.5 (Pin_5), J9.5 (Pin_5), R11.1, R17.1, R19.1, R22.1, R23.1, R24.1, R5.1, R7.1, R8.1, U1.14 (~{RESET}), U1.3 (VCCIO), U3.14 (~{RESET}), U3.3 (VCCIO), U4.2 (3V3), U6.2 (VO), U7.2 (3V3), U8.16 (VCC); no longer C8.1, L1.2
- net +5V: now also C8.1, L1.2, C11.1, J6.A4 (VBUS), J6.A9 (VBUS), J6.B4 (VBUS), J6.B9 (VBUS), J7.A4 (VBUS), J7.A9 (VBUS), J7.B4 (VBUS), J7.B9 (VBUS), J8.1 (Pin_1), J9.1 (Pin_1), U1.15 (VCC), U3.15 (VCC), U5.4 (FB), U6.3 (VI); no longer C4.2
- net EA_00: now also U4.18 (GPIO20)
- net EA_01: now also U4.20 (GPIO22)
- net EA_10: now also U7.18 (GPIO20)
- net EA_11: now also U7.20 (GPIO22)
- net EA_20: now also U4.12 (GPIO11)
- net EA_21: now also U4.16 (GPIO18)
- net EA_30: now also U7.12 (GPIO11)
- net EA_31: now also U7.16 (GPIO18)
- net EB_00: now also U4.19 (GPIO21)
- net EB_01: now also U4.21 (GPIO23)
- net EB_10: now also U7.19 (GPIO21)
- net EB_11: now also U7.21 (GPIO23)
- net EB_20: now also U4.23 (GPIO15)
- net EB_21: now also U4.17 (GPIO19)
- net EB_30: now also U7.23 (GPIO15)
- net EB_31: now also U7.17 (GPIO19)
- net GND: now also C4.2, C1.2, C10.2, C11.2, C12.2, C13.2, C14.2, C15.2, C16.2, C17.2, C2.2, C3.2, C5.2, C9.2, D2.1 (K), D3.1 (K), D4.1 (K), D5.1 (K), J6.A1 (GND), J6.A12 (GND), J6.B1 (GND), J6.B12 (GND), J6.S1 (SHIELD), J7.A1 (GND), J7.A12 (GND), J7.B1 (GND), J7.B12 (GND), J7.S1 (SHIELD), J8.2 (Pin_2), J9.2 (Pin_2), R10.2, R12.2, R13.2, R9.2, SW1.1 (A), SW2.1 (A), SW3.1 (A), SW4.1 (A), U1.16 (GND), U1.6 (GND), U3.16 (GND), U3.6 (GND), U4.1 (GND), U4.28 (GND), U4.29 (GND), U5.6 (GND), U6.1 (GND), U7.1 (GND), U7.28 (GND), U7.29 (GND), U8.8 (GND); no longer C4.1
- net INA_00: now also U4.8 (GPIO0/ADC1_CH0/XTAL_32K_P)
- net INA_01: now also U4.27 (GPIO2/ADC1_CH2)
- net INA_10: now also U7.8 (GPIO0/ADC1_CH0/XTAL_32K_P)
- net INA_11: now also U7.27 (GPIO2/ADC1_CH2)
- net INA_20: now also U4.4 (MTMS/GPIO4/ADC1_CH4)
- net INA_21: now also U4.6 (MTCK/GPIO6/ADC1_CH6)
- net INA_30: now also U7.4 (MTMS/GPIO4/ADC1_CH4)
- net INA_31: now also U7.6 (MTCK/GPIO6/ADC1_CH6)
- net INB_00: now also U4.9 (GPIO1/ADC1_CH1/XTAL_32K_N)
- net INB_01: now also U4.26 (GPIO3/ADC1_CH3)
- net INB_10: now also U7.9 (GPIO1/ADC1_CH1/XTAL_32K_N)
- net INB_11: now also U7.26 (GPIO3/ADC1_CH3)
- net INB_20: now also U4.5 (MTDI/GPIO5/ADC1_CH5)
- net INB_21: now also U4.7 (MTDO/GPIO7)
- net INB_30: now also U7.5 (MTDI/GPIO5/ADC1_CH5)
- net INB_31: now also U7.7 (MTDO/GPIO7)
- net SCL: now also R19.2, R8.2, U4.13 (GPIO12/USB_D-), U7.13 (GPIO12/USB_D-)
- net SDA: now also R17.2, R7.2, U4.14 (GPIO13/USB_D+), U7.14 (GPIO13/USB_D+)
- net SW_00: now also U8.4 (P0)
- net SW_01: now also U8.5 (P1)
- net SW_10: now also U8.6 (P2)
- net SW_11: now also U8.7 (P3)
- net SW_20: now also U8.9 (P4)
- net SW_21: now also U8.10 (P5)
- net SW_30: now also U8.11 (P6)
- net SW_31: now also U8.12 (P7)
- net at R6.2: now also U5.5 (ON/~{OFF})
- net at C7.1, D1.1 (K), L1.1: now also U5.8 (VSW)
- net at C7.2: now also U5.1 (CB)
- new net: R2.2, U1.11 (USBDP)
- new net: Q4.1 (B), R26.2
- new net: D4.2 (A), R16.2
- new net: R24.2, U8.13 (NINT)
- new net: R22.2, U8.15 (SDA)
- new net: R1.2, U1.12 (USBDM)
- new net: J6.A5 (CC1), R10.1
- new net: D5.2 (A), R18.2
- new net: R3.2, U3.12 (USBDM)
- new net: D3.2 (A), R15.2
- new net: D2.2 (A), R14.2
- new net: R4.2, U3.11 (USBDP)
- new net: Q3.1 (B), R25.2
- new net: Q1.1 (B), R20.2
- new net: J6.B5 (CC2), R9.1
- new net: Q2.1 (B), R21.2
- new net: R23.2, U8.14 (SCL)
- new net: J7.A5 (CC1), R13.1
- new net: J7.B5 (CC2), R12.1
- new net BOOT0: C17.1, Q4.3 (C), SW4.2 (B), U4.15 (GPIO9)
- new net BOOT1: C15.1, Q2.3 (C), SW2.2 (B), U7.15 (GPIO9)
- new net DTR0: Q4.2 (E), R25.1, U1.1 (~{DTR})
- new net DTR1: Q2.2 (E), R20.1, U3.1 (~{DTR})
- new net EN0: C16.1, C5.1, Q3.3 (C), R5.2, SW3.2 (B), U4.3 (EN/CHIP_PU)
- new net EN1: C12.1, C14.1, Q1.3 (C), R11.2, SW1.2 (B), U7.3 (EN/CHIP_PU)
- new net LED00: R14.1, U4.10 (GPIO8)
- new net LED01: R15.1, U4.11 (GPIO10)
- new net LED10: R16.1, U7.10 (GPIO8)
- new net LED11: R18.1, U7.11 (GPIO10)
- new net RTS0: Q3.2 (E), R26.1, U1.2 (~{RTS})
- new net RTS1: Q1.2 (E), R21.1, U3.2 (~{RTS})
- new net RX0: J8.4 (Pin_4), U1.20 (TXD), U4.24 (U0RXD/GPIO17)
- new net RX1: J9.4 (Pin_4), U3.20 (TXD), U7.24 (U0RXD/GPIO17)
- new net TX0: J8.3 (Pin_3), U1.4 (RXD), U4.25 (U0TXD/GPIO16)
- new net TX1: J9.3 (Pin_3), U3.4 (RXD), U7.25 (U0TXD/GPIO16)
- new net USB_DM0: J6.A7 (D-), J6.B7 (D-), R1.1
- new net USB_DM1: J7.A7 (D-), J7.B7 (D-), R3.1
- new net USB_DP0: J6.A6 (D+), J6.B6 (D+), R2.1
- new net USB_DP1: J7.A6 (D+), J7.B6 (D+), R4.1
- no-connect marks 11 -> 29
Other:
- note added: "Boot/Reset Buttons"
- note added: "Debug LEDs"
- note added: "ESP32_0"
- note added: "ESP32_1"
- note added: "I2C Expander"
- note added: "UART Ports"
- note added: "USB to UART"
- note added: "USB-C Ports"
- note removed: "Encoder ESP32"
- note removed: "MUX"
- note removed: "Main ESP32"
- moved on the sheet: C6, C7, C8, D1, J?, L1, R6, U2
